File: tapegyseg.sch (KiCad schematic (older format))
At the start: 64 parts, among them J7 line_in, Q1 yjl2301c, Q2 BC817, U12 max1649, U13 H11L1, U14 L79L05_SOT89, U15 L78L33_SOT89

Commit message: Krisztián megjegyzései 1
Parts:
- removed C51: 10u, Capacitor_THT:CP_Radial_D10.0mm_P5.00mm, symbol Device:C_Polarized
- removed D15: do-214AC, Diode_SMD:D_SMA_Handsoldering, symbol Diode:1N4004
- removed R111, R92: 7k2, Resistor_SMD:R_1206_3216Metric_Pad1.30x1.75mm_HandSolder, symbol Device:R
- added C51: 330n, Capacitor_SMD:C_1206_3216Metric_Pad1.33x1.80mm_HandSolder, symbol Device:C
- added D15: 5V6, Diode_SMD:D_MiniMELF_Handsoldering, symbol Device:D_Zener
- C50: value 100n -> 560p; footprint Capacitor_THT:C_Rect_L18.0mm_W6.0mm_P15.00mm_FKS3_FKP3 -> Capacitor_SMD:C_1206_3216Metric_Pad1.33x1.80mm_HandSolder
- D14: value do-214AC -> bzd27c100; footprint Diode_SMD:D_SMA_Handsoldering -> Diode_SMD:D_MELF_Handsoldering
- D16: value do-214AC -> ll4148
- R106, R107, R108, R109, R90, R91: value 7k2 -> 82k
- R110: value 7k2 -> 470k
- R96: value 1k -> 220
Connections:
- net at R91.1: now also Q2.3 (C), C51.2, D15.1 (K); no longer C50.1
- net at D16.1 (K), Q2.1 (B): now also C50.2, D14.1 (K), R110.2
- net at D16.2 (A): now also C50.1, R110.1, R96.2, C51.1, D15.2 (A); no longer Q2.2 (E)
- new net: Q2.2 (E), U13.1
Other:
- moved on the sheet: C50, D16, Q2, R110, R96
Changed lines of the file:
@@
 $Descr A4 11693 8268
 encoding utf-8
-Sheet 7 7
+Sheet 3 7
 Title ""
 Date ""
@@
 P 2100 5200
 F 0 "R90" H 1950 5150 50  0000 C CNN
-F 1 "7k2" H 1950 5250 50  0000 C CNN
+F 1 "82k" H 1950 5250 50  0000 C CNN
 F 2 "Resistor_SMD:R_1206_3216Metric_Pad1.30x1.75mm_HandSolder" V 2030 5200 50  0001 C CNN
 F 3 "~" H 2100 5200 50  0001 C CNN
@@
 P 1700 5200
 F 0 "R91" H 1550 5150 50  0000 C CNN
-F 1 "7k2" H 1550 5250 50  0000 C CNN
+F 1 "82k" H 1550 5250 50  0000 C CNN
 F 2 "Resistor_SMD:R_1206_3216Metric_Pad1.30x1.75mm_HandSolder" V 1630 5200 50  0001 C CNN
 F 3 "~" H 1700 5200 50  0001 C CNN
@@
 L Diode:1N4004 D16
 U 1 1 5F747EE4
-P 3600 5850
-F 0 "D16" H 3600 6067 50  0000 C CNN
-F 1 "do-214AC" H 3600 5976 50  0000 C CNN
-F 2 "Diode_SMD:D_SMA_Handsoldering" H 3600 5675 50  0001 C CNN
-F 3 "http://www.vishay.com/docs/88503/1n4001.pdf" H 3600 5850 50  0001 C CNN
-	1    3600 5850
-	1    0    0    1
-$EndComp
-$Comp
-L Diode:1N4004 D15
-U 1 1 5F748621
-P 3100 5850
-F 0 "D15" H 3100 6067 50  0000 C CNN
-F 1 "do-214AC" H 3100 5976 50  0000 C CNN
-F 2 "Diode_SMD:D_SMA_Handsoldering" H 3100 5675 50  0001 C CNN
-F 3 "http://www.vishay.com/docs/88503/1n4001.pdf" H 3100 5850 50  0001 C CNN
-	1    3100 5850
-	1    0    0    1
+P 3350 5350
+F 0 "D16" H 3350 5567 50  0000 C CNN
+F 1 "ll4148" H 3350 5476 50  0000 C CNN
+F 2 "Diode_SMD:D_SMA_Handsoldering" H 3350 5175 50  0001 C CNN
+F 3 "http://www.vishay.com/docs/88503/1n4001.pdf" H 3350 5350 50  0001 C CNN
+	1    3350 5350
+	0    1    1    0
 $EndComp
 $Comp
@@
 P 2500 5150
 F 0 "D14" H 2500 4933 50  0000 C CNN
-F 1 "do-214AC" H 2500 5024 50  0000 C CNN
-F 2 "Diode_SMD:D_SMA_Handsoldering" H 2500 4975 50  0001 C CNN
+F 1 "bzd27c100" H 2500 5024 50  0000 C CNN
+F 2 "Diode_SMD:D_MELF_Handsoldering" H 2500 4975 50  0001 C CNN
 F 3 "http://www.vishay.com/docs/88503/1n4001.pdf" H 2500 5150 50  0001 C CNN
 	1    2500 5150
@@
 L Device:C C50
 U 1 1 5F749E5D
-P 2750 5500
-F 0 "C50" H 2865 5546 50  0000 L CNN
-F 1 "100n" H 2865 5455 50  0000 L CNN
-F 2 "Capacitor_THT:C_Rect_L18.0mm_W6.0mm_P15.00mm_FKS3_FKP3" H 2788 5350 50  0001 C CNN
-F 3 "~" H 2750 5500 50  0001 C CNN
-	1    2750 5500
-	1    0    0    1
-$EndComp
-Wire Wire Line
-	2750 5150 2750 5350
-$Comp
-L Device:R R92
-U 1 1 5F750076
-P 3450 5600
-F 0 "R92" V 3450 5150 50  0000 L CNN
-F 1 "7k2" V 3450 4900 50  0000 L CNN
-F 2 "Resistor_SMD:R_1206_3216Metric_Pad1.30x1.75mm_HandSolder" V 3380 5600 50  0001 C CNN
-F 3 "~" H 3450 5600 50  0001 C CNN
-	1    3450 5600
-	0    -1   1    0
-$EndComp
-$Comp
-L Device:C_Polarized C51
-U 1 1 5F750A8B
-P 4550 5550
-F 0 "C51" H 4432 5504 50  0000 R CNN
-F 1 "10u" H 4432 5595 50  0000 R CNN
-F 2 "Capacitor_THT:CP_Radial_D10.0mm_P5.00mm" H 4588 5400 50  0001 C CNN
-F 3 "~" H 4550 5550 50  0001 C CNN
-	1    4550 5550
-	-1   0    0    -1
+P 3100 5350
+F 0 "C50" H 3000 5000 50  0000 L CNN
+F 1 "560p" H 2950 5100 50  0000 L CNN
+F 2 "Capacitor_SMD:C_1206_3216Metric_Pad1.33x1.80mm_HandSolder" H 3138 5200 50  0001 C CNN
+F 3 "~" H 3100 5350 50  0001 C CNN
+	1    3100 5350
+	-1   0    0    1
 $EndComp
 $Comp
 L Transistor_BJT:BC817 Q2
 U 1 1 5F751F2C
-P 4950 5950
-F 0 "Q2" V 5278 5950 50  0000 C CNN
-F 1 "BC817" V 5187 5950 50  0000 C CNN
-F 2 "Package_TO_SOT_SMD:SOT-23" H 5150 5875 50  0001 L CIN
-F 3 "https://www.onsemi.com/pub/Collateral/BC818-D.pdf" H 4950 5950 50  0001 L CNN
-	1    4950 5950
-	0    1    -1   0
-$EndComp
-Wire Wire Line
-	2950 5850 2750 5850
-Wire Wire Line
-	3250 5850 3350 5850
-Connection ~ 3350 5850
-Wire Wire Line
-	3350 5850 3450 5850
-Wire Wire Line
-	4550 5150 4550 5400
+P 2750 5750
+F 0 "Q2" V 3078 5750 50  0000 C CNN
+F 1 "BC817" V 2987 5750 50  0000 C CNN
+F 2 "Package_TO_SOT_SMD:SOT-23" H 2950 5675 50  0001 L CIN
+F 3 "https://www.onsemi.com/pub/Collateral/BC818-D.pdf" H 2750 5750 50  0001 L CNN
+	1    2750 5750
+	0    -1   1    0
+$EndComp
 $Comp
 L Device:R R96
 U 1 1 5F7653BC
-P 5500 5850
-F 0 "R96" V 5293 5850 50  0000 C CNN
-F 1 "1k" V 5384 5850 50  0000 C CNN
-F 2 "Resistor_SMD:R_0805_2012Metric_Pad1.20x1.40mm_HandSolder" V 5430 5850 50  0001 C CNN
-F 3 "~" H 5500 5850 50  0001 C CNN
-	1    5500 5850
+P 5700 5650
+F 0 "R96" V 5493 5650 50  0000 C CNN
+F 1 "220" V 5584 5650 50  0000 C CNN
+F 2 "Resistor_SMD:R_0805_2012Metric_Pad1.20x1.40mm_HandSolder" V 5630 5650 50  0001 C CNN
+F 3 "~" H 5700 5650 50  0001 C CNN
+	1    5700 5650
 	0    1    -1   0
 $EndComp
-Wire Wire Line
-	3350 5850 3350 6150
-Wire Wire Line
-	4550 5700 4550 5850
-Connection ~ 4550 5850
-Wire Wire Line
-	4550 5850 4750 5850
-Wire Wire Line
-	5150 5850 5350 5850
 $Comp
 L Isolator:H11L1 U13
@@
 	1    0    0    -1
 $EndComp
-Wire Wire Line
-	4550 5150 5850 5150
-Wire Wire Line
-	5850 5150 5850 5450
-Connection ~ 4550 5150
-Wire Wire Line
-	5850 5650 5850 5850
-Wire Wire Line
-	5850 5850 5650 5850
 $Comp
 L power:GNDD #PWR0160
@@
 	1    0    0    -1
 $EndComp
-Wire Wire Line
-	2650 5150 2750 5150
-Connection ~ 2750 5150
 $Comp
 L Connector:TestPoint TP17
@@
 P 1700 4900
 F 0 "R109" H 1450 4950 50  0000 L CNN
-F 1 "7k2" H 1500 4850 50  0000 L CNN
+F 1 "82k" H 1500 4850 50  0000 L CNN
 F 2 "Resistor_SMD:R_1206_3216Metric_Pad1.30x1.75mm_HandSolder" V 1630 4900 50  0001 C CNN
 F 3 "~" H 1700 4900 50  0001 C CNN
@@
 P 1700 4600
 F 0 "R108" H 1450 4650 50  0000 L CNN
-F 1 "7k2" H 1500 4550 50  0000 L CNN
+F 1 "82k" H 1500 4550 50  0000 L CNN
 F 2 "Resistor_SMD:R_1206_3216Metric_Pad1.30x1.75mm_HandSolder" V 1630 4600 50  0001 C CNN
 F 3 "~" H 1700 4600 50  0001 C CNN
@@
 P 2100 4900
 F 0 "R107" H 2200 4950 50  0000 L CNN
-F 1 "7k2" H 2200 4850 50  0000 L CNN
+F 1 "82k" H 2200 4850 50  0000 L CNN
 F 2 "Resistor_SMD:R_1206_3216Metric_Pad1.30x1.75mm_HandSolder" V 2030 4900 50  0001 C CNN
 F 3 "~" H 2100 4900 50  0001 C CNN
@@
 P 2100 4600
 F 0 "R106" H 2200 4650 50  0000 L CNN
-F 1 "7k2" H 2200 4550 50  0000 L CNN
+F 1 "82k" H 2200 4550 50  0000 L CNN
 F 2 "Resistor_SMD:R_1206_3216Metric_Pad1.30x1.75mm_HandSolder" V 2030 4600 50  0001 C CNN
 F 3 "~" H 2100 4600 50  0001 C CNN
@@
 	1    0    0    -1
 $EndComp
-Wire Wire Line
-	2750 5150 3700 5150
-$Comp
-L Device:R R111
-U 1 1 5F7E91EF
-P 3450 5450
-F 0 "R111" V 3450 5850 50  0000 C CNN
-F 1 "7k2" V 3450 6100 50  0000 C CNN
-F 2 "Resistor_SMD:R_1206_3216Metric_Pad1.30x1.75mm_HandSolder" V 3380 5450 50  0001 C CNN
-F 3 "~" H 3450 5450 50  0001 C CNN
-	1    3450 5450
-	0    1    1    0
-$EndComp
 $Comp
 L Device:R R110
 U 1 1 5F7E9E70
-P 3450 5300
-F 0 "R110" V 3450 5700 50  0000 C CNN
-F 1 "7k2" V 3450 5950 50  0000 C CNN
-F 2 "Resistor_SMD:R_1206_3216Metric_Pad1.30x1.75mm_HandSolder" V 3380 5300 50  0001 C CNN
-F 3 "~" H 3450 5300 50  0001 C CNN
-	1    3450 5300
-	0    1    1    0
-$EndComp
-Wire Wire Line
-	3350 5850 3350 5700
-Wire Wire Line
-	3350 5700 3300 5700
-Wire Wire Line
-	3300 5700 3300 5600
-Wire Wire Line
-	3600 5600 3600 5450
-Wire Wire Line
-	3300 5450 3300 5300
-Wire Wire Line
-	3600 5300 3700 5300
-Wire Wire Line
-	3700 5300 3700 5150
+P 3700 5300
+F 0 "R110" H 3550 5250 50  0000 C CNN
+F 1 "470k" H 3550 5350 50  0000 C CNN
+F 2 "Resistor_SMD:R_1206_3216Metric_Pad1.30x1.75mm_HandSolder" V 3630 5300 50  0001 C CNN
+F 3 "~" H 3700 5300 50  0001 C CNN
+	1    3700 5300
+	-1   0    0    1
+$EndComp
 $Comp
 L Transformer:TEZ2.0-D-2 TR1
@@
 NoConn ~ 3400 1800
 Wire Wire Line
-	3700 5150 4550 5150
-Connection ~ 3700 5150
-Wire Wire Line
-	3350 6150 4950 6150
-Wire Wire Line
-	3750 5850 4550 5850
-Wire Wire Line
 	2200 4000 2200 3950
 Wire Wire Line
@@
 	2100 5400 2100 5350
 Wire Wire Line
-	2750 5650 2750 5850
-Wire Wire Line
-	2750 5850 1700 5850
-Wire Wire Line
 	1700 5350 1700 5850
-Connection ~ 2750 5850
 Connection ~ 6700 5550
 Wire Wire Line
@@
 Wire Wire Line
 	6450 5550 6700 5550
+Wire Wire Line
+	2750 5550 2750 5150
+Wire Wire Line
+	2750 5150 2650 5150
+Wire Wire Line
+	2550 5850 2400 5850
+Wire Wire Line
+	2750 5150 3100 5150
+Wire Wire Line
+	3100 5150 3100 5200
+Connection ~ 2750 5150
+Wire Wire Line
+	3350 5200 3350 5150
+Wire Wire Line
+	3350 5150 3100 5150
+Connection ~ 3100 5150
+$Comp
+L Device:D_Zener D15
+U 1 1 5F8B763B
+P 3350 5650
+F 0 "D15" V 3396 5570 50  0000 R CNN
+F 1 "5V6" V 3305 5570 50  0000 R CNN
+F 2 "Diode_SMD:D_MiniMELF_Handsoldering" H 3350 5650 50  0001 C CNN
+F 3 "~" H 3350 5650 50  0001 C CNN
+	1    3350 5650
+	0    -1   -1   0
+$EndComp
+Wire Wire Line
+	3350 5850 3350 5800
+Wire Wire Line
+	3100 5500 3350 5500
+Connection ~ 3350 5500
+Wire Wire Line
+	3350 5500 3700 5500
+Wire Wire Line
+	3700 5500 3700 5450
+Wire Wire Line
+	3700 5150 3350 5150
+Connection ~ 3350 5150
+$Comp
+L Device:C C51
+U 1 1 5F8CC05D
+P 3700 5650
+F 0 "C51" H 3815 5696 50  0000 L CNN
+F 1 "330n" H 3815 5605 50  0000 L CNN
+F 2 "Capacitor_SMD:C_1206_3216Metric_Pad1.33x1.80mm_HandSolder" H 3738 5500 50  0001 C CNN
+F 3 "~" H 3700 5650 50  0001 C CNN
+	1    3700 5650
+	1    0    0    -1
+$EndComp
+Connection ~ 3700 5500
+Wire Wire Line
+	3350 5850 3700 5850
+Wire Wire Line
+	3700 5850 3700 5800
+Wire Wire Line
+	2400 5850 2400 6250
+Wire Wire Line
+	2400 6250 3350 6250
+Wire Wire Line
+	3350 6250 3350 5850
+Connection ~ 2400 5850
+Wire Wire Line
+	2400 5850 1700 5850
+Connection ~ 3350 5850
+Wire Wire Line
+	2950 5850 3150 5850
+Wire Wire Line
+	3150 5850 3150 6050
+Wire Wire Line
+	3150 6050 4300 6050
+Wire Wire Line
+	4300 6050 4300 5450
+Wire Wire Line
+	4300 5450 5850 5450
+Wire Wire Line
+	3700 5500 4250 5500
+Wire Wire Line
+	4250 5500 4250 5650
+Wire Wire Line
+	4250 5650 5550 5650
 $EndSCHEMATC
